File: KiCad/Daikin.kicad_pcb (KiCad board)
At the start: 2 copper layers, 13.2 x 19.5 mm, 19 parts, among them J1 SPOX, J2 Prog, Q3 PMF250XNEX, U1 ESP32-PICO-MINI-02, U2 LMR16006+FB

Commit message: Tweak prog
Parts:
- J2: footprint Connector_PinHeader_2.54mm:PinHeader_1x05_P2.54mm_Vertical -> RevK:Shelly
- moved J2 5.08 mm to (100.0, 56.4), turned to 0 degrees
Other:
- board text removed: "0"
- board text removed: "3.3V"
- board text removed: "Rx"
- board text removed: "Tx"
Changed lines of the file:
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@@
     )
   )
-  (footprint "Connector_PinHeader_2.54mm:PinHeader_1x05_P2.54mm_Vertical" (layer "B.Cu")
-    (at 105.08 56.4 90)
-    (descr "Through hole straight pin header, 1x05, 2.54mm pitch, single row")
-    (tags "Through hole pin header THT 1x05 2.54mm single row")
-    (property "Sheetfile" "Daikin.kicad_sch")
-    (property "Sheetname" "")
-    (property "exclude_from_bom" "")
-    (attr through_hole exclude_from_bom)
-    (fp_text reference "J2" (at 0 2.33 270) (layer "B.SilkS") hide
+  (footprint "RevK:Shelly" (layer "B.Cu")
+    (at 100 56.4)
+    (property "Sheetfile" "Daikin.kicad_sch")
+    (property "Sheetname" "")
+    (attr through_hole)
+    (fp_text reference "J2" (at 0 2.6 180 unlocked) (layer "B.SilkS") hide
       (effects (font (size 1 1) (thickness 0.15)) (justify mirror))
     )
-    (fp_text value "Prog" (at 0 -12.49 270) (layer "B.Fab")
+    (fp_text value "Prog" (at 0.2 -3.7 180 unlocked) (layer "B.Fab") hide
       (effects (font (size 1 1) (thickness 0.15)) (justify mirror))
     )
-    (fp_text user "${REFERENCE}" (at 0 -5.08) (layer "B.Fab")
+    (fp_text user "↑" (at -2.54 1.27 180 unlocked) (layer "B.SilkS")
+      (effects (font (size 0.5 0.5) (thickness 0.08)) (justify mirror))
+    )
+    (fp_text user "⏚" (at 5.08 1.27 180 unlocked) (layer "B.SilkS")
+      (effects (font (size 0.5 0.5) (thickness 0.08)) (justify mirror))
+    )
+    (fp_text user "↓" (at -5.08 1.27 180 unlocked) (layer "B.SilkS")
+      (effects (font (size 0.5 0.5) (thickness 0.08)) (justify mirror))
+    )
+    (fp_text user "0" (at 2.54 1.27 180 unlocked) (layer "B.SilkS")
+      (effects (font (size 0.5 0.5) (thickness 0.08)) (justify mirror))
+    )
+    (fp_text user "3V3" (at 0 1.27 180 unlocked) (layer "B.SilkS")
+      (effects (font (size 0.5 0.5) (thickness 0.08)) (justify mirror))
+    )
+    (fp_text user "${REFERENCE}" (at 0 2.6) (layer "B.Fab")
       (effects (font (size 1 1) (thickness 0.15)) (justify mirror))
     )
-    (fp_line (start 1.27 1.27) (end 1.27 -11.43) (layer "B.Fab") (width 0.1))
-    (fp_line (start 1.27 -11.43) (end -1.27 -11.43) (layer "B.Fab") (width 0.1))
-    (fp_line (start -1.27 0.635) (end -0.635 1.27) (layer "B.Fab") (width 0.1))
-    (fp_line (start -0.635 1.27) (end 1.27 1.27) (layer "B.Fab") (width 0.1))
-    (fp_line (start -1.27 -11.43) (end -1.27 0.635) (layer "B.Fab") (width 0.1))
-    (pad "1" thru_hole rect (at 0 0 90) (size 1.7 1.7) (drill 1) (layers *.Cu *.Mask)
-      (net 1 "GND") (pinfunction "Pin_1") (pintype "power_in"))
-    (pad "2" thru_hole oval (at 0 -2.54 90) (size 1.7 1.7) (drill 1) (layers *.Cu *.Mask)
-      (net 25 "GPIO0") (pinfunction "Pin_2") (pintype "passive"))
-    (pad "3" thru_hole oval (at 0 -5.08 90) (size 1.7 1.7) (drill 1) (layers *.Cu *.Mask)
-      (net 34 "+3V3") (pinfunction "Pin_3") (pintype "power_in"))
-    (pad "4" thru_hole oval (at 0 -7.62 90) (size 1.7 1.7) (drill 1) (layers *.Cu *.Mask)
-      (net 36 "I") (pinfunction "Pin_4") (pintype "passive"))
-    (pad "5" thru_hole oval (at 0 -10.16 90) (size 1.7 1.7) (drill 1) (layers *.Cu *.Mask)
-      (net 37 "O") (pinfunction "Pin_5") (pintype "passive"))
+    (pad "1" thru_hole rect (at 5.08 0 90) (size 1.7 1.7) (drill 1) (layers *.Cu *.Mask)
+      (net 1 "GND") (pinfunction "GND") (pintype "power_in"))
+    (pad "2" thru_hole oval (at 2.54 0 90) (size 1.7 1.7) (drill 1) (layers *.Cu *.Mask)
+      (net 25 "GPIO0") (pinfunction "0") (pintype "output"))
+    (pad "3" thru_hole oval (at 0 0 90) (size 1.7 1.7) (drill 1) (layers *.Cu *.Mask)
+      (net 34 "+3V3") (pinfunction "3V3") (pintype "power_in"))
+    (pad "4" thru_hole oval (at -2.54 0 90) (size 1.7 1.7) (drill 1) (layers *.Cu *.Mask)
+      (net 36 "I") (pinfunction "Rx") (pintype "output"))
+    (pad "5" thru_hole oval (at -5.08 0 90) (size 1.7 1.7) (drill 1) (layers *.Cu *.Mask)
+      (net 37 "O") (pinfunction "Tx") (pintype "input"))
   )
   (footprint "RevK:Hidden" (layer "B.Cu")
@@
     (effects (font (size 0.5 0.5) (thickness 0.08)) (justify mirror))
   )
-  (gr_text "GND" (at 105.1 55.2) (layer "B.SilkS")
-    (effects (font (size 0.5 0.5) (thickness 0.08)) (justify mirror))
-  )
-  (gr_text "3.3V" (at 100 55.2) (layer "B.SilkS")
-    (effects (font (size 0.5 0.5) (thickness 0.08)) (justify mirror))
-  )
   (gr_text "Daikin" (at 94.4 48.4 90) (layer "B.SilkS")
     (effects (font (size 0.75 0.75) (thickness 0.1)) (justify mirror))
@@
     (effects (font (size 0.5 0.5) (thickness 0.08)) (justify mirror))
   )
-  (gr_text "Tx" (at 94.9 55.2) (layer "B.SilkS")
-    (effects (font (size 0.5 0.5) (thickness 0.08)) (justify mirror))
-  )
-  (gr_text "0" (at 102.55 55.2) (layer "B.SilkS")
-    (effects (font (size 0.5 0.5) (thickness 0.08)) (justify mirror))
-  )
-  (gr_text "Rx" (at 97.45 55.2) (layer "B.SilkS")
-    (effects (font (size 0.5 0.5) (thickness 0.08)) (justify mirror))
-  )
