File: PCB/FaikinDev/Faikin.kicad_pcb (KiCad board)
At the start: 2 copper layers, 70 x 70 mm, 31 parts, among them J1 1x5, J2 TC2030-USB-NL, J3 Reset, Q1 BSS138PS, U1 TPS562243, U4 ESP32-S3-MINI-1

Commit message: Tweaks
Parts:
- added C1: 100nF, RevK:C_0201, F.Cu at (138.0, 64.6)
- moved R8 0.42 mm to (138.3, 65.6), turned to 180 degrees
Routing:
- net GND: track 1.05 -> 2.51 mm, vias 45 -> 50
- net +3.3V: track 45.9 -> 46.7 mm
- net DC: track 37.2 -> 37.8 mm
- net SW: track 10.00 -> 10.5 mm

Commit message: Tweak
Parts:
- moved L1 0.30 mm to (141.2, 70.2)
- moved C16 0.10 mm to (138.1, 68.4)
Routing:
- net DC: track 37.4 -> 39.0 mm
- net GND: vias 50 -> 51
