File: PCB/Faikout/Faikout.kicad_sch (KiCad schematic)
At the start: 47 parts, among them J1 1x5, J2 TC2030-USB-NL, J3 Reset, Q1 BSS138PS, U1 TPS562246, U4 ESP32-S3-MINI-1

Commit message: Rename
Other:
- title: Faikin -> Faikout
Changed lines of the file:
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@@
 	(paper "A4")
 	(title_block
-		(title "Faikin")
+		(title "Faikout")
 		(rev "1")
 		(comment 1 "@TheRealRevK")
